Commit message: Apply joint calibration: zero offsets, ±60° joint limit (driver, URDF, gait)
Measured stops: joint1 -70/+95 deg, joints 2-6 about +/-100 deg. 60 deg keeps a
10 deg margin on the tightest (joint1 negative side).

Co-Authored-By: Claude Opus 5.5 <noreply@anthropic.com>

File: ros2_ws/src/snakebot_description/urdf/snakebot.urdf.xacro (robot description, xacro)
@@ -24,5 +24,5 @@
   <xacro:property name="m_lidar" value="0.185"/>      <!-- YDLIDAR G2 datasheet -->
   <!-- ===== Joints (XM430-W350 @ 12 V: 4.1 N·m stall, 46 rpm no-load) ===== -->
-  <xacro:property name="joint_limit" value="${pi/2}"/>   <!-- TODO: set to where the brackets actually collide -->
+  <xacro:property name="joint_limit" value="${radians(60)}"/>  <!-- stops measured 2026-10-05: joint1 -70/+95 deg, joints 2-6 ~+/-100 deg; 10 deg margin on the tightest -->
   <xacro:property name="joint_effort" value="4.1"/>
   <xacro:property name="joint_velocity" value="4.8"/>     <!-- rad/s -->

Commit message: Verify joint 1 direction against URDF with the lidar; note joint1 collision
Co-Authored-By: Claude Opus 5.5 <noreply@anthropic.com>

File: ros2_ws/src/snakebot_description/urdf/snakebot.urdf.xacro (robot description, xacro)
@@ -24,5 +24,5 @@
   <xacro:property name="m_lidar" value="0.185"/>      <!-- YDLIDAR G2 datasheet -->
   <!-- ===== Joints (XM430-W350 @ 12 V: 4.1 N·m stall, 46 rpm no-load) ===== -->
-  <xacro:property name="joint_limit" value="${radians(60)}"/>  <!-- stops measured 2026-10-05: joint1 -70/+95 deg, joints 2-6 ~+/-100 deg; 10 deg margin on the tightest -->
+  <xacro:property name="joint_limit" value="${radians(60)}"/>  <!-- stops measured 2026-10-05: joint1 -70 (seg1 hits the lidar UART adapter) / +95 deg, joints 2-6 ~+/-100 deg; 10 deg margin on the tightest -->
   <xacro:property name="joint_effort" value="4.1"/>
   <xacro:property name="joint_velocity" value="4.8"/>     <!-- rad/s -->
